File: doc/HomeBoard.brd (EAGLE design)
At the start: 65 x 35 mm, 39 parts, among them IC1 L6981, Q5 BSS138, Q6 BSS138, U1 ESP32-WROOM-32D

Commit message: updated1603
Parts:
- added R13: 10k, #AK-Library:0603
- R1: value (none) -> 140k
- R2: value (none) -> 47k
- R4: value (none) -> 22R
- moved PAD1 1.55 mm to (40.1, 21.1)
- moved PAD2 1.55 mm to (38.9, 21.1)
- moved PAD3 1.30 mm to (40.1, 23.4)
- moved PAD4 1.30 mm to (38.9, 23.4)
Connections:
- net 3.3V: now also R13.2
- net GPIO18: now also R13.1
Routing:
- net 3.3V: track 19.6 -> 25.4 mm
- net GPIO0: track 14.8 -> 16.8 mm
- net GPIO18: track 14.4 -> 16.0 mm
- net CH3: track 27.5 -> 28.9 mm

Commit message: Update HomeBoard.brd
Parts:
- D1: value (none) -> LTST-S220TBKT
Changed lines of the file:
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@@
 <attribute name="VALUE" x="12.192" y="22.352" size="0.8128" layer="27" font="vector" ratio="15" align="top-center"/>
 </element>
-<element name="D1" library="#AK-Library" library_urn="urn:adsk.eagle:library:17478144" package="LED-ANGLE-2MM" package3d_urn="urn:adsk.eagle:package:34599462/2" value="" x="24.892" y="1.016" smashed="yes" rot="R90">
+<element name="D1" library="#AK-Library" library_urn="urn:adsk.eagle:library:17478144" package="LED-ANGLE-2MM" package3d_urn="urn:adsk.eagle:package:34599462/2" value="LTST-S220TBKT" x="24.892" y="1.016" smashed="yes" rot="R90">
 <attribute name="NAME" x="27.2805" y="1.048" size="0.7112" layer="25" font="vector" ratio="15" rot="R270" align="bottom-center"/>
 <attribute name="VALUE" x="25.8445" y="1.016" size="0.6096" layer="27" font="vector" ratio="20" rot="R90" align="top-center"/>
