File: doc/HomeBoard.sch (EAGLE design)
At the start: 39 parts, among them IC1 L6981, Q5 BSS138, Q6 BSS138, U1 ESP32-WROOM-32D

Commit message: updated1603
Parts:
- added R13: 10k, #AK-Library:RESISTOR0603
- R1: value (none) -> 140k
- R2: value (none) -> 47k
- R4: value (none) -> 22R
Connections:
- net 3.3V: now also R13.2
- net GPIO18: now also R13.1
Other:
- moved on the sheet: C5
Changed lines of the file:
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@@
 <part name="GND1" library="SparkFun-PowerSymbols" library_urn="urn:adsk.eagle:library:530" deviceset="GND" device=""/>
 <part name="SUPPLY2" library="SparkFun-PowerSymbols" library_urn="urn:adsk.eagle:library:530" deviceset="VCC" device=""/>
-<part name="S1" library="#AK-Library" library_urn="urn:adsk.eagle:library:17478144" deviceset="MOMENTARY-SWITCH-SPST" device="-PTH-RIGHT-ANGLE-KIT" package3d_urn="urn:adsk.eagle:package:34599795/3"/>
+<part name="S1" library="#AK-Library" library_urn="urn:adsk.eagle:library:17478144" deviceset="MOMENTARY-SWITCH-SPST" device="-PTH-RIGHT-ANGLE-KIT" package3d_urn="urn:adsk.eagle:package:34599795/4"/>
 <part name="IC1" library="#AK-Library" library_urn="urn:adsk.eagle:library:17478144" deviceset="L6981" device="" package3d_urn="urn:adsk.eagle:package:34599460/2"/>
 <part name="J1" library="#Connectors" library_urn="urn:adsk.eagle:library:17281549" deviceset="CONN_02" device="5MM" package3d_urn="urn:adsk.eagle:package:17403359/6"/>
@@
 <part name="C4" library="#AK-Library" library_urn="urn:adsk.eagle:library:17478144" deviceset="CAP" device="-0603" package3d_urn="urn:adsk.eagle:package:16984038/3" value="0.1uF"/>
 <part name="L1" library="#AK-Library" library_urn="urn:adsk.eagle:library:17478144" deviceset="INDUCTOR" device="-7.3X6.6" package3d_urn="urn:adsk.eagle:package:34599461/2"/>
-<part name="R1" library="#AK-Library" library_urn="urn:adsk.eagle:library:17478144" deviceset="RESISTOR" device="0603" package3d_urn="urn:adsk.eagle:package:16984038/3" value=" "/>
-<part name="R2" library="#AK-Library" library_urn="urn:adsk.eagle:library:17478144" deviceset="RESISTOR" device="0603" package3d_urn="urn:adsk.eagle:package:16984038/3" value=" "/>
+<part name="R1" library="#AK-Library" library_urn="urn:adsk.eagle:library:17478144" deviceset="RESISTOR" device="0603" package3d_urn="urn:adsk.eagle:package:16984038/3" value="140k"/>
+<part name="R2" library="#AK-Library" library_urn="urn:adsk.eagle:library:17478144" deviceset="RESISTOR" device="0603" package3d_urn="urn:adsk.eagle:package:16984038/3" value="47k"/>
 <part name="SUPPLY3" library="SparkFun-PowerSymbols" library_urn="urn:adsk.eagle:library:530" deviceset="VCC" device=""/>
 <part name="GND2" library="SparkFun-PowerSymbols" library_urn="urn:adsk.eagle:library:530" deviceset="GND" device=""/>
@@
 <part name="D1" library="#AK-Library" library_urn="urn:adsk.eagle:library:17478144" deviceset="LED" device="-ANGLE-2MM" package3d_urn="urn:adsk.eagle:package:34599462/2"/>
 <part name="GND7" library="SparkFun-PowerSymbols" library_urn="urn:adsk.eagle:library:530" deviceset="GND" device=""/>
-<part name="R4" library="#AK-Library" library_urn="urn:adsk.eagle:library:17478144" deviceset="RESISTOR" device="0603" package3d_urn="urn:adsk.eagle:package:16984038/3" value=" "/>
+<part name="R4" library="#AK-Library" library_urn="urn:adsk.eagle:library:17478144" deviceset="RESISTOR" device="0603" package3d_urn="urn:adsk.eagle:package:16984038/3" value="22R"/>
 <part name="GND8" library="SparkFun-PowerSymbols" library_urn="urn:adsk.eagle:library:530" deviceset="GND" device=""/>
 <part name="SUPPLY6" library="SparkFun-PowerSymbols" library_urn="urn:adsk.eagle:library:530" deviceset="VCC" device=""/>
@@
 <part name="GND15" library="SparkFun-PowerSymbols" library_urn="urn:adsk.eagle:library:530" deviceset="GND" device=""/>
 <part name="EN" library="#AK-Library" library_urn="urn:adsk.eagle:library:17478144" deviceset="MOMENTARY-SWITCH-SPST" device="-SMD-6.0X3.5MM" package3d_urn="urn:adsk.eagle:package:34599812/2"/>
+<part name="R13" library="#AK-Library" library_urn="urn:adsk.eagle:library:17478144" deviceset="RESISTOR" device="0603" package3d_urn="urn:adsk.eagle:package:16984038/3" value="10k"/>
+<part name="SUPPLY12" library="SparkFun-PowerSymbols" library_urn="urn:adsk.eagle:library:530" deviceset="3.3V" device=""/>
 </parts>
 <sheets>
@@
 <attribute name="VALUE" x="96.52" y="162.814" size="1.778" layer="96" align="bottom-center"/>
 </instance>
-<instance part="C5" gate="G$1" x="104.14" y="104.14" smashed="yes">
-<attribute name="NAME" x="104.902" y="105.41" size="1.27" layer="95" font="vector"/>
-<attribute name="VALUE" x="106.426" y="103.378" size="1.27" layer="96" font="vector" rot="R270"/>
-</instance>
-<instance part="SUPPLY5" gate="G$1" x="111.76" y="111.76" smashed="yes">
-<attribute name="VALUE" x="111.76" y="114.554" size="1.778" layer="96" align="bottom-center"/>
-</instance>
-<instance part="GND4" gate="1" x="111.76" y="93.98" smashed="yes">
-<attribute name="VALUE" x="111.76" y="93.726" size="1.778" layer="96" align="top-center"/>
+<instance part="C5" gate="G$1" x="104.14" y="101.6" smashed="yes">
+<attribute name="NAME" x="104.902" y="102.87" size="1.27" layer="95" font="vector"/>
+<attribute name="VALUE" x="104.902" y="98.806" size="1.27" layer="96" font="vector"/>
+</instance>
+<instance part="SUPPLY5" gate="G$1" x="104.14" y="111.76" smashed="yes">
+<attribute name="VALUE" x="104.14" y="114.554" size="1.778" layer="96" align="bottom-center"/>
+</instance>
+<instance part="GND4" gate="1" x="104.14" y="93.98" smashed="yes">
+<attribute name="VALUE" x="104.14" y="93.726" size="1.778" layer="96" align="top-center"/>
 </instance>
 <instance part="C6" gate="G$1" x="22.86" y="93.98" smashed="yes">
@@
 <instance part="EN" gate="G$1" x="132.08" y="91.44" smashed="yes">
 <attribute name="NAME" x="132.08" y="92.964" size="1.778" layer="95" font="vector" align="bottom-center"/>
+</instance>
+<instance part="R13" gate="G$1" x="226.06" y="68.58" smashed="yes">
+<attribute name="NAME" x="226.06" y="71.374" size="1.27" layer="95" font="vector" align="bottom-center"/>
+<attribute name="VALUE" x="226.06" y="69.85" size="1.016" layer="96" font="vector" rot="R180" align="top-center"/>
+</instance>
+<instance part="SUPPLY12" gate="G$1" x="231.14" y="71.12" smashed="yes">
+<attribute name="VALUE" x="231.14" y="73.914" size="1.778" layer="96" align="bottom-center"/>
 </instance>
 </instances>
@@
 <segment>
 <pinref part="C5" gate="G$1" pin="1"/>
-<wire x1="104.14" y1="101.6" x2="104.14" y2="99.06" width="0.1524" layer="91"/>
-<wire x1="104.14" y1="99.06" x2="111.76" y2="99.06" width="0.1524" layer="91"/>
-<wire x1="111.76" y1="99.06" x2="111.76" y2="101.6" width="0.1524" layer="91"/>
 <pinref part="GND4" gate="1" pin="GND"/>
-<wire x1="111.76" y1="99.06" x2="111.76" y2="96.52" width="0.1524" layer="91"/>
-<junction x="111.76" y="99.06"/>
+<wire x1="104.14" y1="99.06" x2="104.14" y2="96.52" width="0.1524" layer="91"/>
 </segment>
 <segment>
@@
 <pinref part="U1" gate="G$1" pin="3V3"/>
 <wire x1="88.9" y1="109.22" x2="104.14" y2="109.22" width="0.1524" layer="91"/>
-<wire x1="104.14" y1="109.22" x2="111.76" y2="109.22" width="0.1524" layer="91"/>
-<wire x1="111.76" y1="109.22" x2="111.76" y2="106.68" width="0.1524" layer="91"/>
 <pinref part="C5" gate="G$1" pin="2"/>
-<wire x1="104.14" y1="106.68" x2="104.14" y2="109.22" width="0.1524" layer="91"/>
+<wire x1="104.14" y1="104.14" x2="104.14" y2="109.22" width="0.1524" layer="91"/>
 <junction x="104.14" y="109.22"/>
 <pinref part="SUPPLY5" gate="G$1" pin="3.3V"/>
-<wire x1="111.76" y1="111.76" x2="111.76" y2="109.22" width="0.1524" layer="91"/>
-<junction x="111.76" y="109.22"/>
+<wire x1="104.14" y1="111.76" x2="104.14" y2="109.22" width="0.1524" layer="91"/>
 </segment>
 <segment>
@@
 <wire x1="43.18" y1="25.4" x2="43.18" y2="30.48" width="0.1524" layer="91"/>
 </segment>
+<segment>
+<pinref part="R13" gate="G$1" pin="2"/>
+<wire x1="228.6" y1="68.58" x2="231.14" y2="68.58" width="0.1524" layer="91"/>
+<wire x1="231.14" y1="68.58" x2="231.14" y2="71.12" width="0.1524" layer="91"/>
+<pinref part="SUPPLY12" gate="G$1" pin="3.3V"/>
+</segment>
 </net>
 <net name="EN" class="0">
@@
 <label x="223.52" y="55.88" size="1.27" layer="95" rot="R180" xref="yes"/>
 </segment>
-</net>
+<segment>
+<pinref part="R13" gate="G$1" pin="1"/>
+<wire x1="223.52" y1="68.58" x2="220.98" y2="68.58" width="0.1524" layer="91"/>
+<label x="220.98" y="68.58" size="1.27" layer="95" rot="R180" xref="yes"/>
+</segment>
+</net>

Commit message: Update HomeBoard.sch
Parts:
- D1: value (none) -> LTST-S220TBKT
Changed lines of the file:
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@@
 <part name="Q6" library="#AK-Library" library_urn="urn:adsk.eagle:library:17478144" deviceset="MOSFET-N" device="-SOT23-3" package3d_urn="urn:adsk.eagle:package:17233478/4" value="BSS138"/>
 <part name="GND6" library="SparkFun-PowerSymbols" library_urn="urn:adsk.eagle:library:530" deviceset="GND" device=""/>
-<part name="D1" library="#AK-Library" library_urn="urn:adsk.eagle:library:17478144" deviceset="LED" device="-ANGLE-2MM" package3d_urn="urn:adsk.eagle:package:34599462/2"/>
+<part name="D1" library="#AK-Library" library_urn="urn:adsk.eagle:library:17478144" deviceset="LED" device="-ANGLE-2MM" package3d_urn="urn:adsk.eagle:package:34599462/2" value="LTST-S220TBKT"/>
 <part name="GND7" library="SparkFun-PowerSymbols" library_urn="urn:adsk.eagle:library:530" deviceset="GND" device=""/>
 <part name="R4" library="#AK-Library" library_urn="urn:adsk.eagle:library:17478144" deviceset="RESISTOR" device="0603" package3d_urn="urn:adsk.eagle:package:16984038/3" value="22R"/>
@@
 <instance part="D1" gate="D1" x="132.08" y="58.42" smashed="yes" rot="R90">
 <attribute name="NAME" x="136.652" y="54.991" size="1.778" layer="95" font="vector" rot="R180"/>
-<attribute name="VALUE" x="136.652" y="60.325" size="1.778" layer="96" font="vector" rot="R180" align="top-left"/>
+<attribute name="VALUE" x="130.048" y="61.595" size="1.778" layer="96" font="vector" align="top-left"/>
 </instance>
 <instance part="GND7" gate="1" x="139.7" y="50.8" smashed="yes">
